File: pcb/efr32mg21_devboard/efr32mg21_devboard.kicad_pcb (KiCad board)
At the start: 2 copper layers, 40 x 40 mm, 37 parts, among them CON1 CORTEX-DEBUGGER, J1 Conn_01x10, J2 microusb, J3 Conn_01x10, J4 Conn_02x02_Counter_Clockwise, J5 Conn_02x02_Counter_Clockwise, SW1 SW_Push, SW2 SW_Push, U1 EFR32MG21A020F768IM32-BR, U2 TLV70033_SOT23-5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

Commit message: breakout board
Other:
- board text added: "EFR32MG21"
